File: circuit-stuff/cansat wiring v2.sch (EAGLE design)
At the start: 6 parts

Commit message: Add files via upload
Parts:
- removed RFM9X_LORA_RADIO: (no value), con-lstb:MA09-1
- added 1000UF: (no value), capacitor-wima:C2.5/2
- added HC12: (no value), con-lstb:MA05-1
- renumbered 3.3V_REGULATOR to 5V_REGULATOR
Connections:
- removed net N$11: ARDUINO_NANO1.A4, BME680.6
- removed net N$12: ARDUINO_NANO1.A5, BME680.5
- net +: now also 1000UF.2, ARDUINO_NANO1.GND@1, HC12.2, POWER.1; no longer POWER.2, RFM9X_LORA_RADIO.2
- net -: now also POWER.2; no longer POWER.1
- net N$1: now also ARDUINO_NANO1.D9, BME680.4; no longer ARDUINO_NANO1.D5, RFM9X_LORA_RADIO.9
- net N$2: now also ARDUINO_NANO1.D11, BME680.5; no longer ARDUINO_NANO1.D4, RFM9X_LORA_RADIO.8
- net N$4: now also 1000UF.1, HC12.1; no longer RFM9X_LORA_RADIO.1
- net N$6: now also ARDUINO_NANO1.D12, BME680.6; no longer ARDUINO_NANO1.D11, RFM9X_LORA_RADIO.7
- net N$7: now also ARDUINO_NANO1.D5, HC12.4; no longer ARDUINO_NANO1.D12, RFM9X_LORA_RADIO.6
- net N$8: now also ARDUINO_NANO1.D10, BME680.7; no longer ARDUINO_NANO1.D13, RFM9X_LORA_RADIO.5
- net N$9: now also ARDUINO_NANO1.D4, HC12.3; no longer ARDUINO_NANO1.D9, RFM9X_LORA_RADIO.4
